File: Hardware/ETHERBEAR.sch (EAGLE design)
At the start: 95 parts, among them IC1 MC33269DT-5.0, IC2 CP2102N-A01-GQFN24, IC4 LM358D, IC5 ATMEGA328P TQFP32, IC6 W6100-LQFP, IC7 MCP24AA025E48, J1 DC_2_1MM, J2 USB-C-16P-16P, P2 ICSP:MAIN, P4 microSD, Q1 FDN340P, Q2 2N7002, U1 HY931147C-RJ45

Commit message: Schematic changes for ATmega1284P
Parts:
- removed A6, A7: M01, SuperHouse-Connectors:M01-PLAIN
- removed C28, C30, C31: 100nF, SuperHouse-DiscreteSemi:CAP0603
- removed C29: 100nF 0603, SuperHouse-DiscreteSemi:CAP0603
- removed H1: Digital_8_13, SuperHouse-Connectors:M10-SOCKET
- removed H2: Power, SuperHouse-Connectors:M08-SOCKET
- removed IC7: MCP24AA025E48, freetronics-jon:MCP24AA025E48
- removed LED10: D13/RED, SuperHouse-LEDs:LED0603
- removed P2: ICSP:MAIN, SuperHouse-Connectors:ICSP-PIN
- removed R12: 22.1K, SuperHouse-DiscreteSemi:RESISTOR0603
- removed R13: 47.5K, SuperHouse-DiscreteSemi:RESISTOR0603
- removed R14: 4K7, SuperHouse-DiscreteSemi:RESISTOR0603
- removed RN8: 2K2, SuperHouse-DiscreteSemi:4R-NCAY16
- removed SJ6, SJ7: SJC, SuperHouse-Jumpers:SJC-NORMAL
- removed U$17, U$19: CRYSTAL-GND3X2, SuperHouse-Oscillators:CRYSTAL-GND3X2
- added C11, C12, C8: 100nF, SuperHouse-DiscreteSemi:CAP0603
- added C2: 10uF 6.3V A TANT, SuperHouse-DiscreteSemi:CAP_POL1206
- added IC3: LM358D, linear:LM358D
- added J5: DC_2_1MM, SuperHouse-Connectors:POWER_JACK-SLOTS
- added J6: USB-C-16P-16P, SuperHouse-Connectors:USB-C-16P-16P
- added J7: INTERRUPT, SuperHouse-Connectors:M01-PLAIN
- added J9: ICSP, SuperHouse-Connectors:ICSP-PIN
- added LED1: PWR/BLUE, SuperHouse-LEDs:LED0603
- added R4: 12K 1%, SuperHouse-DiscreteSemi:RESISTOR0603
- added R5: 300R 1%, SuperHouse-DiscreteSemi:RESISTOR0603
- added RN7: 2K2, SuperHouse-DiscreteSemi:4R-NCAY16
- added SJ1: RESET-EN, SuperHouse-Jumpers:SJC-NORMAL
- added XTL1: 25MHz, SuperHouse-Oscillators:CRYSTAL-GND3X2
- added XTL2: 16MHz, SuperHouse-Oscillators:CRYSTAL-GND3X2
- C1: value 100nF 0603 -> 10uF 6.3V A TANT; device SuperHouse-DiscreteSemi:CAP0603 -> SuperHouse-DiscreteSemi:CAP_POL1206
- C10, C13: value 10uF 6.3V A TANT -> 100nF; device SuperHouse-DiscreteSemi:CAP_POL1206 -> SuperHouse-DiscreteSemi:CAP0603
- C14, C19: value 100nF 0603 -> 100nF
- C15, C16: value 13pF -> 100nF
- C20, C21: value 22pF 0603 -> 100nF
- C24, C25: value 100nF -> 13pF
- C26: value 100nF -> 22pF
- C27: value 100nF 0603 -> 22pF
- C7: value 100nF 0603 -> 1uF
- C9: value 1uF 0603 -> 100nF
- IC4: value LM358D -> W6100-LQFP; device linear:LM358D -> SuperHouse-ICs:W6100-LQFP
- IC5: value ATMEGA328P TQFP32 -> MCP24AA025E48; device SuperHouse-MCUs:ATMEGA8-AI -> freetronics-jon:MCP24AA025E48
- IC6: value W6100-LQFP -> ATMEGA1284P-TQFP; device SuperHouse-ICs:W6100-LQFP -> SuperHouse-MCUs:ATMEGA1284P-TQFP
- J1: value DC_2_1MM -> Digital_8_13; device SuperHouse-Connectors:POWER_JACK-SLOTS -> SuperHouse-Connectors:M10-SOCKET
- J2: value USB-C-16P-16P -> Power; device SuperHouse-Connectors:USB-C-16P-16P -> SuperHouse-Connectors:M08-SOCKET
- LED2: value PWR/BLUE -> YELLOW
- LED3: value YELLOW -> RED
- LED4: value RED -> TX/YEL
- LED5: value TX/YEL -> RX/GRN
- LED6: value RX/GRN -> GREEN
- LED8: value GREEN -> YELLOW
- LED9: value YELLOW -> D13/RED
- R6: value 12K 1% -> 1K
- R7: value 300R 1% -> 22.1K
- R8: value 1K 0603 -> 47.5K
- R9: value 10K -> 4K7
- RN1, RN2: value 330R -> 1K
- SJ3: value RESET-EN -> SJC
- SJ4: value MODE -> SJC; device SuperHouse-Jumpers:SJ-NORMAL -> SuperHouse-Jumpers:SJC-NORMAL
- renumbered H3 to J3, H4 to J4, IC1 to REG1, JP3 to J8, L4 to L3, P4 to J10, R15 to R10, U1 to J11, VR1 to REG2, VR2 to REG3
Connections:
- removed net A0: IC5.PC0(ADC0), J3.1
- removed net A1: IC5.PC1(ADC1), J3.2
- removed net A2: IC5.PC2(ADC2), J3.3
- removed net A3: IC5.PC3(ADC3), J3.4
- removed net A4_SDA: H1.9, IC5.PC4(ADC4/SDA), J3.5, SJ5.1
- removed net A5_SCL: H1.10, IC5.PC5(ADC5/SCL), J3.6, SJ6.1
- removed net D11_MOSI: H1.4, IC5.PB3(MOSI/OC2), IC6.MOSI, P2.4, RN6C.2
- removed net D12_MISO: H1.5, IC5.PB4(MISO), IC6.MISO, J10.DO, P2.1
- removed net D2: IC5.PD2(INT0), J4.3
- removed net D3: IC5.PD3(INT1), J4.4
- removed net MODE: IC6.MOD0, R3.2, SJ4.1
- removed net N$21: A7.1, IC5.ADC7
- removed net N$22: A6.1, IC5.ADC6
- removed net N$37: IC6.!INT, R9.1
- new net A0_D14: IC6.PA7(ADC7/PCINT7), J3.1
- new net A1_D15: IC6.PA6(ADC6/PCINT6), J3.2
- new net A2_D16: IC6.PA5(ADC5/PCINT5), J3.3
- new net A3_D17: IC6.PA4(ADC4/PCINT4), J3.4
- new net A4_D18: IC6.PA3(ADC3/PCINT3), J3.5
- new net A5_D19: IC6.PA2(ADC2/PCINT2), J3.6
- new net D10_SS: IC6.PB4(PCINT12/OC0B/!SS!)
- new net D11_COPI: IC4.MOSI, IC6.PB5(PCINT13/ICP3/MOSI), J1.4, J9.4, RN6C.2
- new net D12_CIPO: IC4.MISO, IC6.PB6(PCINT14/OC3A/MISO), J1.5, J10.DO, J9.1
- new net D2_RX1: IC6.PD2(PCINT26/RXD1/INT0), J4.3
- new net D3_TX1: IC6.PD3(PCINT27/TXD1/INT1), J4.4
- new net N$9: IC4.!INT, J7.1, R3.2
- new net SCL: IC6.PC0(SCL/PCINT16), J1.10, SJ4.1
- new net SDA: IC6.PC1(SDA/PCINT17), J1.9, SJ3.1
- net 1V2A: now also C1.+, C11.1, IC4.1V2A; no longer C17.1, C4.+, IC6.1V2A
- net 1V2D: now also C15.1, C2.+, C20.1, C22.1, C23.1, IC4.1V2D; no longer C26.1, C28.1, C3.+, C30.1, C31.1, IC6.1V2D
- net 1V2O: now also IC4.1V2O; no longer IC6.1V2O
- net 3.3V: now also C21.1, C4.+, IC3A.-IN, IC4.3V3D, J2.4, LED2.A; no longer C10.+, C29.1, H2.4, IC4A.-IN, IC6.3V3D, LED9.A, R9.2, SJ4.2
- net 3V3A: now also C12.1, C14.1, C19.1, C3.+, IC4.3V3A; no longer C13.+, C18.1, C22.1, C25.1, IC6.3V3A
- net 5V: now also C10.1, C16.1, IC3P.V+, IC5.VCC, IC6.AVCC, IC6.VCC, J2.2, J2.5, J9.2, LED1.A, LED9.A, R3.1, R7.2, R9.1; no longer C14.1, C27.1, H2.2, H2.5, IC4P.V+, IC5.AVCC, IC5.VCC@1, IC5.VCC@2, IC7.VCC, LED10.A, LED2.A, P2.2, R12.2, R14.1
- net ACTLED: now also IC4.!ACT; no longer IC6.!ACT
- net AREF: now also C8.1, IC6.AREF, J1.8; no longer C1.1, H1.8, IC5.AREF
- net COLLED: now also IC4.!COL; no longer IC6.!COL
- net D+: now also J6.D+; no longer J2.D+
- net D-: now also J6.D-; no longer J2.D-
- net D0_RX: now also IC6.PD0(PCINT24/RXD0/T3); no longer IC5.PD0(RXD)
- net D10_CS: now also IC4.!CS, J1.3; no longer H1.3, IC5.PB2(SS/OC1B), IC6.!CS
- net D13_SCK: now also IC4.SCLK, IC6.PB7(PCINT15/OC3B/SCK), J1.6, J9.3; no longer H1.6, IC5.PB5(SCK), IC6.SCLK, P2.3
- net D1_TX: now also IC6.PD1(PCINT25/TXD0); no longer IC5.PD1(TXD)
- net D4: now also IC6.PB0(PCINT8/XCK0/T0), SJ5.2; no longer IC5.PD4(XCK/T0), SJ7.2
- net D5: now also IC6.PB1(PCINT9/CLKO/T1); no longer IC5.PD5(T1)
- net D6: now also IC6.PB2(PCINT10/INT2/AIN0); no longer IC5.PD6(AIN0)
- net D7: now also IC6.PB3(PCINT11/OC0A/AIN1); no longer IC5.PD7(AIN1)
- net D8: now also IC6.PD5(PCINT29/OC1A), J1.1; no longer H1.1, IC5.PB0(ICP)
- net D9: now also IC6.PD6(PCINT30/OC2B/ICP), J1.2; no longer H1.2, IC5.PB1(OC1A)
- net DTR: now also SJ1.1; no longer SJ3.1
- net FDXLED: now also IC4.!DPX; no longer IC6.!DPX
- net GND: now also C1.-, C10.2, C11.2, C12.2, C19.2, C2.-, C20.2, C21.2, C26.1, C27.1, C8.2, IC3P.V-, IC4.GND, IC4.GNDA, IC4.MOD0, IC4.MOD1, IC4.MOD2, IC4.MOD3, IC5.A0, IC5.A1, IC5.GND, J1.7, J2.6, J2.7, J5.GND, J5.GNDBREAK, J6.GND, J9.6, R5.2, R8.1, RN7A.1, RN7B.1, RN7C.1, XTL1.GND, XTL2.GND; no longer C1.2, C10.-, C13.-, C20.1, C21.1, C26.2, C27.2, C28.2, C29.2, C30.2, C31.2, H1.7, H2.6, H2.7, IC4P.V-, IC5.AGND, IC5.GND@1, IC5.GND@2, IC6.GNDA, IC6.MOD1, IC6.MOD2, IC6.MOD3, IC7.A0, IC7.A1, IC7.GND, J1.GND, J1.GNDBREAK, J2.GND, P2.6, R13.1, R3.1, R7.2, RN8A.1, RN8B.1, RN8C.1, U$17.GND, U$17.GND2, U$19.GND, U$19.GND2
- net LINKLED: now also IC4.!LINK; no longer IC6.!LINK
- net N$1: now also C18.1; no longer C24.1
- net N$10: now also J6.CC2; no longer J2.CC2
- net N$11: now also LED5.C; no longer LED6.C
- net N$115: now also J6.VBUS; no longer J2.VBUS
- net N$12: now also IC3A.+IN; no longer IC4A.+IN
- net N$13: now also LED4.C; no longer LED5.C
- net N$14: now also LED1.C; no longer LED2.C
- net N$18: now also IC3B.-IN, IC3B.OUT; no longer IC4B.-IN, IC4B.OUT
- net N$19: now also IC3A.OUT, IC3B.+IN; no longer IC4A.OUT, IC4B.+IN
- net N$2: now also C26.2, IC6.XTAL1, XTL2.1; no longer C20.2, IC5.PB6(XTAL1/TOSC1), U$19.XTL1
- net N$20: now also RN7A.2; no longer RN8A.2
- net N$24: now also RN7B.2; no longer RN8B.2
- net N$25: now also RN7C.2; no longer RN8C.2
- net N$26: now also LED7.C; no longer LED8.C
- net N$27: now also SJ5.1; no longer SJ7.1
- net N$28: now also LED8.C; no longer LED9.C
- net N$29: now also IC5.SDA, R9.2, SJ3.2; no longer IC7.SDA, R14.2, SJ5.2
- net N$3: now also C13.1, SJ1.2; no longer C19.1, SJ3.2
- net N$30: now also C24.1, IC4.XSCO, XTL1.2; no longer C15.1, IC6.XSCO, U$17.XTL1
- net N$32: now also C25.1, IC4.XSCI, XTL1.1; no longer C16.1, IC6.XSCI, U$17.XTL2
- net N$321: now also C17.1; no longer C23.1
- net N$327: now also LED6.C; no longer LED7.C
- net N$329: now also LED2.C; no longer LED3.C
- net N$34: now also J6.CC1; no longer J2.CC1
- net N$35: now also R4.2, R5.1; no longer R6.2, R7.1
- net N$36: now also IC4.RSET_BG, R4.1; no longer IC6.RSET_BG, R6.1
- net N$39: now also R7.1, R8.2; no longer R12.1, R13.2
- net N$4: now also LED9.C, R6.2; no longer LED10.C, R8.2
- net N$5: now also IC5.SCL, SJ4.2; no longer IC7.SCL, SJ6.2
- net N$6: now also R6.1; no longer R8.1
- net N$60: now also J5.PWR; no longer J1.PWR
- net N$7: now also C27.2, IC6.XTAL2, XTL2.2; no longer C21.2, IC5.PB7(XTAL2/TOSC2), U$19.XTL2
- net N$8: now also LED3.C; no longer LED4.C
- net RESET: now also C13.2, IC4.!RESET, J2.3, J9.5; no longer C19.2, H2.3, IC5.PC6(/RESET), P2.5
- net RXIN: now also IC4.RXIN; no longer IC6.RXIN
- net RXIP: now also IC4.RXIP; no longer IC6.RXIP
- net SPDLED: now also IC4.!SPD; no longer IC6.!SPD
- net TXON: now also IC4.TXON; no longer IC6.TXON
- net TXOP: now also IC4.TXOP; no longer IC6.TXOP
- net VIN: now also J2.8; no longer H2.8
Other:
- note added: "ATmega1284P Microcontroller"
- note added: "D13 LED"
- note added: "EtherBear (Arduino compatible with Ethernet)"
- note added: "SKU: EB"
- note added: "SPI CIPO"
- note added: "SPI COPI"
- note added: "SPI SCK"
- note added: "V1.0 (2020-08-06)"
- note added: "W6100 !CS"
- note added: "Wiznet W6100 !INT is an output. The 10K pull-up is included so that if this output is connected to an Arduino pin, it will be biased HIGH and can be used to detect Ethernet activity when pulled LOW."
- note added: "uSD !CS"
- note added: "www.superhouse.tv/eb"
- note removed: "ATmega328P Microcontroller"
- note removed: "EtherUNO (Arduino compatible with Ethernet)"
- note removed: "Open: W6100 (default) Closed: W5500"
- note removed: "SKU: EU"
- note removed: "V4.0 (2020-07-12)"
- note removed: "Wiznet Mode"
- note removed: "www.superhouse.tv/eu"
